File: esp8266-artnet-mini.sch (KiCad schematic (older format))
At the start: 25 parts, among them J1 PWR, J2 DMX, J3 PROG, U1 uA7805, U2 ESP-07S, U3 TLV1117-33, U4 MAX485E

Commit message: Updated project to KiCad 5
Parts:
- C1, C2, C3, C4, C5, C6, C7: symbol C -> Device:C
- J1: symbol Conn_01x02 -> esp8266-artnet-mini-rescue:Conn_01x02
- J2, J3: symbol Conn_01x03 -> esp8266-artnet-mini-rescue:Conn_01x03
- JP1, JP2, JP3: symbol Jumper_NO_Small -> Device:Jumper_NO_Small
- R1, R2, R3, R4, R5, R6, R7, R8: symbol R -> Device:R
- U1: symbol uA7805 -> esp8266-artnet-mini-rescue:uA7805
- U2: symbol ESP-07S -> esp8266-artnet-mini-rescue:ESP-07S
- U3: symbol TLV1117-33 -> esp8266-artnet-mini-rescue:TLV1117-33
- U4: symbol MAX485E -> esp8266-artnet-mini-rescue:MAX485E
